File: mk3/pcb/sw63_mk3.brd (EAGLE design)
At the start: 35 x 35 mm, 62 parts, among them J1 USB-C_2.0_SMT, Q1 LGE2305, Q2 BC817S, Q3 BC817S, SW1 KSC321JLFS, SW2 EVQ-P7J01P, U1 ATSAMD21E18A-MU, U2 DS3231MZ+, U3 TLC5916IPW, U4 TLC5916IPW, U5 TLC5916IPW, U6 MIC5504YM5-TR, U7 MCP73832T-2ACI/OT

Commit message: finishing schematics
Parts:
- removed LD22: LED_SMT_0805, BASTL_LEDS:LED_0805
- added B+, B-: TEST_PIN_LARGE, BASTL_PINHEADERS:TEST_PIN_2.0
- added Q4: TEMT6200FX01, BASTL_TRANZISTORS:TEMT6200FX01
- added R14: 10k, BASTL_RESISTORS:RESISTOR0603
- moved C9 9.12 mm to (20.7, 12.9), turned to 270 degrees
- moved C2 1.95 mm to (17.9, 30.4), turned to 90 degrees
- moved C10 1.26 mm to (12.5, 11.4), turned to 270 degrees
- moved C4 0.52 mm to (21.4, 3.51), turned to 0 degrees
- moved C8 0.50 mm to (15.3, 32.4)
- moved U1 0.18 mm to (16.7, 12.1), turned to 90 degrees
- turned LD1 to 90 degrees
- turned LD10 to 90 degrees
- turned LD11 to 90 degrees
- turned LD12 to 90 degrees
- turned LD2 to 90 degrees
- turned LD3 to 90 degrees
- turned LD4 to 90 degrees
- turned LD5 to 90 degrees
- turned LD6 to 90 degrees
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- renumbered LD13 to PLUS, LD14 to MINUS, LD15 to HOURS, LD16 to MINUTES, LD17 to UP, LD18 to RIGHT, LD19 to DOWN, LD20 to LEFT, LD21 to PM
Connections:
- removed net EP: U1.33
- removed net VDDANA: U1.9
- removed net VDDCORE: U1.29
- removed net VDDIN: U1.30
- new net LIGHT_SENS: Q4.E, R14.2, U1.3
- new net N$20: LD10.C, U3.6
- new net N$25: LD5.C, U3.12
- new net N$26: C9.2, U1.29
- new net N$27: LD4.C, U4.9
- new net N$28: LD3.C, U4.10
- new net N$29: LD2.C, U4.11
- new net N$31: MINUTES.K, U4.8
- new net N$32: HOURS.K, U4.7
- new net N$33: MINUS.K, U4.6
- new net N$34: PLUS.K, U4.5
- new net SCL: R5.2, U1.12, U2.8
- new net SDA: R6.2, U1.11, U2.7
- new net SWCLK: SWD.P$4, U1.31
- new net SWDIO: SWD.P$2, U1.32
- net !CHARGING: now also U1.13
- net !RESET: now also SWD.P$3
- net ACTIVE: now also Q4.C, U1.4
- net BAT: now also B+.P$1
- net BRIGHT: now also U1.19
- net BTN: now also U1.1
- net CLK: now also U1.8
- net D+: now also U1.25
- net D-: now also U1.24
- net DAT: now also U1.7
- net GND: now also B-.P$1, C10.1, C11.1, C9.1, R14.1, SWD.P$5, U1.33
- net LAT: now also U1.6
- net N$21: now also LD9.C, U3.5; no longer PLUS.K, U3.7
- net N$22: now also LD8.C, U3.9; no longer MINUS.K, U3.6
- net N$23: now also LD7.C, U3.10; no longer HOURS.K, U3.5
- net N$24: now also LD6.C, U3.11; no longer MINUTES.K, U3.8
- net N$5: now also LD12.C, U3.8; no longer R6.2, U2.7
- net N$7: now also LD11.C, U3.7; no longer R5.2, U2.8
- net VBUS_DTCT: now also U1.5
- net VDD: now also C10.2, C11.2, SWD.P$1, U1.30, U1.9
Routing:
- net N$21: track 16.1 -> 0.00 mm
- net N$30: track 15.9 -> 0.00 mm, vias 1 -> 0
- net N$22: track 8.30 -> 0.00 mm
- net N$24: track 5.43 -> 0.00 mm
- net SCL: track 0.00 -> 5.26 mm
- net N$7: track 5.26 -> 0.00 mm
- net VDDLEDS: track 56.2 -> 51.3 mm, vias 1 -> 0
- net N$33: track 0.00 -> 4.86 mm
- net N$34: track 0.00 -> 4.22 mm
- net SDA: track 0.00 -> 2.88 mm
- net N$5: track 2.88 -> 0.00 mm
- net N$23: track 2.35 -> 0.00 mm
- net !RESET: track 0.00 -> 1.03 mm
- net VDD: track 7.62 -> 7.12 mm

Commit message: routing done
Parts:
- moved C11 2.85 mm to (21.4, 12.4), turned to 270 degrees
- moved C9 2.30 mm to (21.6, 15.0), turned to 0 degrees
- moved C10 1.02 mm to (11.5, 11.2)
- moved R7 0.51 mm to (15.5, 20.5)
- moved C5 0.32 mm to (15.5, 17.7)
- moved C7 0.19 mm to (8.56, 14.5)
- moved R2 0.13 mm to (27.2, 27.6)
- moved B- 0.13 mm to (10.9, 24.8)
- moved R9 0.11 mm to (4.11, 14.0)
- moved R8 0.11 mm to (11.7, 14.5)
- moved C6 0.10 mm to (2.40, 14.0)
Connections:
- net GND: now also U1.21
- net N$31: now also HOURS.K; no longer MINUTES.K
- net N$32: now also MINUTES.K; no longer HOURS.K
Routing:
- net !RESET: track 1.03 -> 81.1 mm, vias 0 -> 4
- net VDDLEDS: track 51.3 -> 115.5 mm, vias 0 -> 6
- net VDD: track 7.12 -> 71.0 mm, vias 0 -> 3
- net GNDLEDS: track 0.00 -> 56.5 mm, vias 0 -> 5
- net LAT: track 0.00 -> 51.7 mm, vias 0 -> 4
- net BAT: track 2.39 -> 42.9 mm, vias 0 -> 2
- net VBUS_DTCT: track 1.34 -> 40.9 mm, vias 0 -> 2
- net SCL: track 5.26 -> 40.0 mm, vias 0 -> 2
- net VBUS_FUSED: track 15.7 -> 50.0 mm, vias 0 -> 2
- net ACTIVE: track 0.00 -> 34.2 mm, vias 0 -> 1
- net CLK: track 0.00 -> 33.8 mm, vias 0 -> 5
- net GND: track 0.00 -> 32.5 mm, vias 0 -> 94
- net SDA: track 2.88 -> 35.3 mm, vias 0 -> 2
- net !CHARGING: track 0.00 -> 27.7 mm, vias 0 -> 2
- net DAT: track 0.00 -> 26.0 mm, vias 0 -> 2
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- added copper zone on layer 1, net GND
- added copper zone on layer 16, net GND
Other:
- board text added: "+"

Commit message: layout tweaks
Routing:
- net GND: vias 94 -> 109
