File: mk3/pcb/sw63_mk3.brd (EAGLE design)
At the start: 35 x 35 mm, 65 parts, among them J1 USB-C_2.0_SMT, Q1 LGE2305, Q2 BC817S, Q3 BC817S, Q4 TEMT6200FX01, SW1 KSC321JLFS, SW2 EVQ-P7J01P, U1 ATSAMD21E18A-MU, U2 DS3231MZ+, U3 TLC5916IPW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

Commit message: board update
Other:
- board size 35 x 35 mm -> 35 x 36 mm
Changed lines of the file:
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@@
 <setting verticaltext="up"/>
 </settings>
-<grid distance="1" unitdist="mil" unit="mil" style="lines" multiple="1" display="yes" altdistance="0.01" altunitdist="mm" altunit="mm"/>
+<grid distance="0.2" unitdist="mm" unit="mm" style="lines" multiple="1" display="yes" altdistance="0.0001" altunitdist="mm" altunit="mm"/>
 <layers>
 <layer number="1" name="Top" color="4" fill="1" visible="yes" active="yes"/>
@@
 <layer number="46" name="Milling" color="3" fill="1" visible="no" active="yes"/>
 <layer number="47" name="Measures" color="7" fill="1" visible="no" active="yes"/>
-<layer number="48" name="Document" color="7" fill="1" visible="no" active="yes"/>
+<layer number="48" name="Document" color="7" fill="1" visible="yes" active="yes"/>
 <layer number="49" name="Reference" color="7" fill="1" visible="no" active="yes"/>
 <layer number="50" name="dxf" color="7" fill="1" visible="no" active="no"/>
@@
 <fusionsync huburn="a.YnVzaW5lc3M6YmFzdGxpbnN0cnVtZW50cw" projecturn="a.YnVzaW5lc3M6YmFzdGxpbnN0cnVtZW50cyNEMjAyMjAzMTQ1MDY5Nzg3MDE" f3durn="urn:adsk.wipprod:dm.lineage:Zd9BFt0GRf6VfhXkAI8fwA" pcbguid="" lastpulledtime="" lastsyncedchangeguid="" latestrevisionid="20768d3f-f369-4c0b-8290-80feba7ce2bf" lastsyncedrevisionid="20768d3f-f369-4c0b-8290-80feba7ce2bf" lastboardhashguid="0b9f5ede-f65d-a811-1811-53758ec48789" lastpushedtime="2024-08-14T12:10:00Z" linktopcb3d="true"/>
 <plain>
-<circle x="17.5" y="17.5" radius="17.5" width="0.000025" layer="20"/>
+<circle x="17.5" y="17.5" radius="17.5" width="0.000025" layer="48"/>
 <hole x="3.5" y="10" drill="1.6"/>
 <hole x="3.5" y="25" drill="1.6"/>
@@
 <vertex x="20.74775" y="27.9004125"/>
 </polygon>
+<wire x1="22" y1="34.4159" x2="22" y2="35.5" width="0.001" layer="20"/>
+<wire x1="22" y1="35.5" x2="13" y2="35.5" width="0.001" layer="20"/>
+<wire x1="13" y1="35.5" x2="13" y2="34.4159" width="0.001" layer="20"/>
+<wire x1="13" y1="0.5841" x2="13" y2="-0.5" width="0.001" layer="20"/>
+<wire x1="13" y1="-0.5" x2="22" y2="-0.5" width="0.001" layer="20"/>
+<wire x1="22" y1="-0.5" x2="22" y2="0.5841" width="0.001" layer="20"/>
+<wire x1="13" y1="0.5841" x2="13" y2="34.4159" width="0.001" layer="20" curve="-150.199611"/>
+<wire x1="22" y1="34.4159" x2="22" y2="0.5841" width="0.001" layer="20" curve="-150.199611"/>
+<polygon width="0.001" layer="41">
+<vertex x="13" y="34.2"/>
+<vertex x="13.3751" y="34.3109" curve="-34.459937"/>
+<vertex x="22.0359" y="34.1961" curve="204.295025"/>
+<vertex x="22.2" y="35.8" curve="-12.611469"/>
+<vertex x="13" y="35.8" curve="192.611647"/>
+</polygon>
+<polygon width="0.001" layer="42">
+<vertex x="13" y="34.2"/>
+<vertex x="13.3751" y="34.3109" curve="-34.459937"/>
+<vertex x="22.0359" y="34.1961" curve="204.295025"/>
+<vertex x="22.2" y="35.8" curve="-12.611469"/>
+<vertex x="13" y="35.8" curve="192.611647"/>
+</polygon>
+<polygon width="0.001" layer="41">
+<vertex x="22" y="0.8"/>
+<vertex x="21.6249" y="0.6891" curve="-34.459937"/>
+<vertex x="12.9641" y="0.8039" curve="204.295025"/>
+<vertex x="12.8" y="-0.8" curve="-12.611469"/>
+<vertex x="22" y="-0.8" curve="192.611647"/>
+</polygon>
+<polygon width="0.001" layer="42">
+<vertex x="22" y="0.8"/>
+<vertex x="21.6249" y="0.6891" curve="-34.459937"/>
+<vertex x="12.9641" y="0.8039" curve="204.295025"/>
+<vertex x="12.8" y="-0.8" curve="-12.611469"/>
+<vertex x="22" y="-0.8" curve="192.611647"/>
+</polygon>
+<circle x="17.5" y="17.5" radius="17.6" width="0.2" layer="22"/>
 </plain>
 <attributes>

Commit message: schematic notes
Connections:
- net N$6 renamed VSEL
Changed lines of the file:
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@@
 <layer number="46" name="Milling" color="3" fill="1" visible="no" active="yes"/>
 <layer number="47" name="Measures" color="7" fill="1" visible="no" active="yes"/>
-<layer number="48" name="Document" color="7" fill="1" visible="yes" active="yes"/>
+<layer number="48" name="Document" color="7" fill="1" visible="no" active="yes"/>
 <layer number="49" name="Reference" color="7" fill="1" visible="no" active="yes"/>
 <layer number="50" name="dxf" color="7" fill="1" visible="no" active="no"/>
@@
 <wire x1="21.69" y1="29.979375" x2="21.69" y2="28.5538" width="0.3048" layer="16"/>
 </signal>
-<signal name="N$6">
+<signal name="VSEL">
 <contactref element="D1" pad="C"/>
 <contactref element="U6" pad="1"/>
