File: mk3/pcb/sw63_mk3_2.sch (EAGLE design)
At the start: 68 parts, among them J1 USB-C_2.0_SMT, Q1 LGE2305, Q2 N-MOSFET, Q4 TEMT6200FX01, SW1 KSC321JLFS, SW2 EVQ-P7J01P, U1 ATSAMD21E18A-MU, U2 DS3231MZ+, U3 TLC5916IPW, U4 TLC5916IPW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

Commit message: 3_2 update
Connections:
- net D+: now also U1.D+/PA25; no longer U1.PA25
- net D-: now also U1.D-/PA24; no longer U1.PA24
- net SWCLK: now also U1.SWCLK/PA30; no longer U1.PA30
- net SWDIO: now also U1.SWDIO/PA31; no longer U1.PA31
Changed lines of the file:
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@@
 <drawing>
 <settings>
-<setting alwaysvectorfont="yes"/>
+<setting alwaysvectorfont="no"/>
 <setting verticaltext="up"/>
 </settings>
@@
 <part name="LD11" library="BASTL_LEDS" library_urn="urn:adsk.eagle:library:32977677" deviceset="LED_SMT" device="_1206" package3d_urn="urn:adsk.eagle:package:45095787/2"/>
 <part name="LD12" library="BASTL_LEDS" library_urn="urn:adsk.eagle:library:32977677" deviceset="LED_SMT" device="_1206" package3d_urn="urn:adsk.eagle:package:45095787/2"/>
-<part name="MINUS" library="BASTL_LEDS" library_urn="urn:adsk.eagle:library:32977677" deviceset="LED_THT" device="-5MM_R" package3d_urn="urn:adsk.eagle:package:45109722/2"/>
-<part name="PLUS" library="BASTL_LEDS" library_urn="urn:adsk.eagle:library:32977677" deviceset="LED_THT" device="-5MM_G" package3d_urn="urn:adsk.eagle:package:45109721/2"/>
-<part name="HOURS" library="BASTL_LEDS" library_urn="urn:adsk.eagle:library:32977677" deviceset="LED_THT" device="-5MM_B" package3d_urn="urn:adsk.eagle:package:45109720/2"/>
-<part name="MINUTES" library="BASTL_LEDS" library_urn="urn:adsk.eagle:library:32977677" deviceset="LED_THT" device="-5MM_Y" package3d_urn="urn:adsk.eagle:package:45109719/2"/>
-<part name="UP" library="BASTL_LEDS" library_urn="urn:adsk.eagle:library:32977677" deviceset="LED_RECT" device="-3.2X2" package3d_urn="urn:adsk.eagle:package:45095773/2"/>
-<part name="RIGHT" library="BASTL_LEDS" library_urn="urn:adsk.eagle:library:32977677" deviceset="LED_RECT" device="-3.2X2" package3d_urn="urn:adsk.eagle:package:45095773/2"/>
-<part name="DOWN" library="BASTL_LEDS" library_urn="urn:adsk.eagle:library:32977677" deviceset="LED_RECT" device="-3.2X2" package3d_urn="urn:adsk.eagle:package:45095773/2"/>
-<part name="LEFT" library="BASTL_LEDS" library_urn="urn:adsk.eagle:library:32977677" deviceset="LED_RECT" device="-3.2X2" package3d_urn="urn:adsk.eagle:package:45095773/2"/>
+<part name="MINUS" library="BASTL_LEDS" library_urn="urn:adsk.eagle:library:32977677" deviceset="LED_THT" device="-5MM_R" package3d_urn="urn:adsk.eagle:package:45109722/3"/>
+<part name="PLUS" library="BASTL_LEDS" library_urn="urn:adsk.eagle:library:32977677" deviceset="LED_THT" device="-5MM_G" package3d_urn="urn:adsk.eagle:package:45109721/3"/>
+<part name="HOURS" library="BASTL_LEDS" library_urn="urn:adsk.eagle:library:32977677" deviceset="LED_THT" device="-5MM_B" package3d_urn="urn:adsk.eagle:package:45109720/3"/>
+<part name="MINUTES" library="BASTL_LEDS" library_urn="urn:adsk.eagle:library:32977677" deviceset="LED_THT" device="-5MM_Y" package3d_urn="urn:adsk.eagle:package:45109719/3"/>
+<part name="UP" library="BASTL_LEDS" library_urn="urn:adsk.eagle:library:32977677" deviceset="LED_RECT" device="-3.2X2" package3d_urn="urn:adsk.eagle:package:45095773/3"/>
+<part name="RIGHT" library="BASTL_LEDS" library_urn="urn:adsk.eagle:library:32977677" deviceset="LED_RECT" device="-3.2X2" package3d_urn="urn:adsk.eagle:package:45095773/3"/>
+<part name="DOWN" library="BASTL_LEDS" library_urn="urn:adsk.eagle:library:32977677" deviceset="LED_RECT" device="-3.2X2" package3d_urn="urn:adsk.eagle:package:45095773/3"/>
+<part name="LEFT" library="BASTL_LEDS" library_urn="urn:adsk.eagle:library:32977677" deviceset="LED_RECT" device="-3.2X2" package3d_urn="urn:adsk.eagle:package:45095773/3"/>
 <part name="PM" library="BASTL_LEDS" library_urn="urn:adsk.eagle:library:32977677" deviceset="LED_THT" device="-3MM_ALT" package3d_urn="urn:adsk.eagle:package:45095771/2"/>
 <part name="SW1" library="BASTL_SWITCHES" library_urn="urn:adsk.eagle:library:32903743" deviceset="KSC3XXJ" device="" package3d_urn="urn:adsk.eagle:package:40210534/2" value="KSC321JLFS"/>
@@
 <segment>
 <wire x1="15.24" y1="-12.7" x2="17.78" y2="-12.7" width="0.1524" layer="91"/>
-<pinref part="U1" gate="G$1" pin="PA25"/>
+<pinref part="U1" gate="G$1" pin="D+/PA25"/>
 <label x="17.78" y="-12.7" size="1.27" layer="95" ratio="15" xref="yes"/>
 </segment>
@@
 <segment>
 <wire x1="15.24" y1="-15.24" x2="17.78" y2="-15.24" width="0.1524" layer="91"/>
-<pinref part="U1" gate="G$1" pin="PA24"/>
+<pinref part="U1" gate="G$1" pin="D-/PA24"/>
 <label x="17.78" y="-15.24" size="1.27" layer="95" ratio="15" xref="yes"/>
 </segment>
@@
 <net name="SWDIO" class="0">
 <segment>
-<pinref part="U1" gate="G$1" pin="PA31"/>
+<pinref part="U1" gate="G$1" pin="SWDIO/PA31"/>
 <wire x1="15.24" y1="-2.54" x2="17.78" y2="-2.54" width="0.1524" layer="91"/>
 <label x="17.78" y="-2.54" size="1.27" layer="95" ratio="12" xref="yes"/>
@@
 <net name="SWCLK" class="0">
 <segment>
-<pinref part="U1" gate="G$1" pin="PA30"/>
+<pinref part="U1" gate="G$1" pin="SWCLK/PA30"/>
 <wire x1="15.24" y1="-5.08" x2="17.78" y2="-5.08" width="0.1524" layer="91"/>
 <label x="17.78" y="-5.08" size="1.27" layer="95" ratio="12" xref="yes"/>

Commit message: 3_2 update
Parts:
- J1: value USB-C_2.0_SMT -> USB-C_2.0_SMT_WS; device BASTL_CONNECTORS:USB-C_2.0_SMT -> BASTL_CONNECTORS:USB-C_2.0_SMT_WS
Connections:
- net GND: now also U1.PA14
Changed lines of the file:
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@@
 <part name="U5" library="BASTL_ICS" library_urn="urn:adsk.eagle:library:32977748" deviceset="TLC5916" device="IPW" package3d_urn="urn:adsk.eagle:package:35867227/3"/>
 <part name="U2" library="BASTL_ICS" library_urn="urn:adsk.eagle:library:32977748" deviceset="DS3231MZ+" device="" package3d_urn="urn:adsk.eagle:package:32977849/5"/>
-<part name="J1" library="BASTL_CONNECTORS" library_urn="urn:adsk.eagle:library:32904192" deviceset="USB-C_2.0_SMT" device="" package3d_urn="urn:adsk.eagle:package:45095758/5"/>
+<part name="J1" library="BASTL_CONNECTORS" library_urn="urn:adsk.eagle:library:32904192" deviceset="USB-C_2.0_SMT_WS" device="" package3d_urn="urn:adsk.eagle:package:45908691/2"/>
 <part name="LD1" library="BASTL_LEDS" library_urn="urn:adsk.eagle:library:32977677" deviceset="LED_SMT" device="_1206" package3d_urn="urn:adsk.eagle:package:45095787/2"/>
 <part name="LD2" library="BASTL_LEDS" library_urn="urn:adsk.eagle:library:32977677" deviceset="LED_SMT" device="_1206" package3d_urn="urn:adsk.eagle:package:45095787/2"/>
@@
 <part name="D4" library="BASTL_DIODES" library_urn="urn:adsk.eagle:library:32977972" deviceset="SCHOTTKY_DIODE" device="_SOD523" package3d_urn="urn:adsk.eagle:package:42502794/4" value="RB521S"/>
 <part name="D5" library="BASTL_DIODES" library_urn="urn:adsk.eagle:library:32977972" deviceset="SCHOTTKY_DIODE" device="_SOD523" package3d_urn="urn:adsk.eagle:package:42502794/4" value="RB521S"/>
+<part name="GND23" library="BASTL_SYMBOLS" library_urn="urn:adsk.eagle:library:32975873" deviceset="GND" device=""/>
 </parts>
 <sheets>
@@
 REPLACE VBUS_FUSED
 WITH VSEL</text>
+<text x="-39.116" y="-34.29" size="1.27" layer="94" ratio="12">Just for layout.</text>
 </plain>
 <instances>
@@
 <attribute name="NAME" x="27.432" y="-33.5534" size="1.778" layer="95"/>
 <attribute name="VALUE" x="27.432" y="-36.0934" size="1.778" layer="96"/>
+</instance>
+<instance part="GND23" gate="1" x="-25.4" y="-38.1" smashed="yes">
+<attribute name="VALUE" x="-27.94" y="-40.64" size="1.778" layer="96"/>
 </instance>
 </instances>
@@
 <pinref part="GND13" gate="1" pin="GND"/>
 </segment>
+<segment>
+<pinref part="GND23" gate="1" pin="GND"/>
+<pinref part="U1" gate="G$1" pin="PA14"/>
+<wire x1="-25.4" y1="-35.56" x2="-25.4" y2="-33.02" width="0.1524" layer="91"/>
+<wire x1="-25.4" y1="-33.02" x2="-20.32" y2="-33.02" width="0.1524" layer="91"/>
+</segment>
 </net>

Commit message: add 3_2 board files
Parts:
- F1: value 500mA -> BSMD0805-050-24V
- J1: value USB-C_2.0_SMT_WS -> GT-USB-7070C
- Q1: value LGE2305 -> 2305
- Q2: value N-MOSFET -> 2302
- SW2: value EVQ-P7J01P -> TSC4A 160gf-WZ 016
- U6: value MIC5504YM5-TR -> ME6211C33M5G-N
Other:
- note removed: "REWORK THIS SECTION: REPLACE VBUS_FUSED WITH VSEL"
Changed lines of the file:
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@@
 <drawing>
 <settings>
-<setting alwaysvectorfont="no"/>
+<setting alwaysvectorfont="yes"/>
 <setting verticaltext="up"/>
 </settings>
@@
 <part name="U5" library="BASTL_ICS" library_urn="urn:adsk.eagle:library:32977748" deviceset="TLC5916" device="IPW" package3d_urn="urn:adsk.eagle:package:35867227/3"/>
 <part name="U2" library="BASTL_ICS" library_urn="urn:adsk.eagle:library:32977748" deviceset="DS3231MZ+" device="" package3d_urn="urn:adsk.eagle:package:32977849/5"/>
-<part name="J1" library="BASTL_CONNECTORS" library_urn="urn:adsk.eagle:library:32904192" deviceset="USB-C_2.0_SMT_WS" device="" package3d_urn="urn:adsk.eagle:package:45908691/2"/>
+<part name="J1" library="BASTL_CONNECTORS" library_urn="urn:adsk.eagle:library:32904192" deviceset="USB-C_2.0_SMT_WS" device="" package3d_urn="urn:adsk.eagle:package:45908691/3" value="GT-USB-7070C"/>
 <part name="LD1" library="BASTL_LEDS" library_urn="urn:adsk.eagle:library:32977677" deviceset="LED_SMT" device="_1206" package3d_urn="urn:adsk.eagle:package:45095787/2"/>
 <part name="LD2" library="BASTL_LEDS" library_urn="urn:adsk.eagle:library:32977677" deviceset="LED_SMT" device="_1206" package3d_urn="urn:adsk.eagle:package:45095787/2"/>
@@
 <part name="PM" library="BASTL_LEDS" library_urn="urn:adsk.eagle:library:32977677" deviceset="LED_THT" device="-3MM_ALT" package3d_urn="urn:adsk.eagle:package:45095771/2"/>
 <part name="SW1" library="BASTL_SWITCHES" library_urn="urn:adsk.eagle:library:32903743" deviceset="KSC3XXJ" device="" package3d_urn="urn:adsk.eagle:package:40210534/2" value="KSC321JLFS"/>
-<part name="U6" library="BASTL_ICS" library_urn="urn:adsk.eagle:library:32977748" deviceset="MIC5504YM5-TR" device="" package3d_urn="urn:adsk.eagle:package:34025889/5"/>
+<part name="U6" library="BASTL_ICS" library_urn="urn:adsk.eagle:library:32977748" deviceset="MIC5504YM5-TR" device="" package3d_urn="urn:adsk.eagle:package:34025889/5" value="ME6211C33M5G-N"/>
 <part name="SWD" library="BASTL_CONNECTORS" library_urn="urn:adsk.eagle:library:32904192" deviceset="2X3POGO" device="NO_VIA" package3d_urn="urn:adsk.eagle:package:32904263/3"/>
 <part name="U7" library="BASTL_ICS" library_urn="urn:adsk.eagle:library:32977748" deviceset="MCP73831T-2ACI" device="" package3d_urn="urn:adsk.eagle:package:34025889/5" value="MCP73832T-2ACI/OT"/>
-<part name="F1" library="BASTL_FUSES" library_urn="urn:adsk.eagle:library:32977952" deviceset="PTC" device="" package3d_urn="urn:adsk.eagle:package:32977962/4" value="500mA"/>
+<part name="F1" library="BASTL_FUSES" library_urn="urn:adsk.eagle:library:32977952" deviceset="PTC" device="" package3d_urn="urn:adsk.eagle:package:32977962/4" value="BSMD0805-050-24V"/>
 <part name="GND1" library="BASTL_SYMBOLS" library_urn="urn:adsk.eagle:library:32975873" deviceset="GND" device=""/>
 <part name="GND2" library="BASTL_SYMBOLS" library_urn="urn:adsk.eagle:library:32975873" deviceset="GND" device=""/>
@@
 <part name="C2" library="BASTL_CAPACITORS" library_urn="urn:adsk.eagle:library:32978038" deviceset="CAPACITOR0805" device="" package3d_urn="urn:adsk.eagle:package:32978071/3" value="10u"/>
 <part name="GND6" library="BASTL_SYMBOLS" library_urn="urn:adsk.eagle:library:32975873" deviceset="GND" device=""/>
-<part name="Q1" library="BASTL_TRANZISTORS" library_urn="urn:adsk.eagle:library:32975847" deviceset="LGE2305" device="" package3d_urn="urn:adsk.eagle:package:32975863/4"/>
+<part name="Q1" library="BASTL_TRANZISTORS" library_urn="urn:adsk.eagle:library:32975847" deviceset="LGE2305" device="" package3d_urn="urn:adsk.eagle:package:32975863/4" value="2305"/>
 <part name="D1" library="BASTL_DIODES" library_urn="urn:adsk.eagle:library:32977972" deviceset="SCHOTTKY_DIODE" device="" package3d_urn="urn:adsk.eagle:package:32978000/2" value="1N5819"/>
 <part name="R4" library="BASTL_RESISTORS" library_urn="urn:adsk.eagle:library:32975925" deviceset="RESISTOR0603" device="" package3d_urn="urn:adsk.eagle:package:32975936/2" value="10k"/>
@@
 <part name="VDDLEDS4" library="BASTL_SYMBOLS" library_urn="urn:adsk.eagle:library:32975873" deviceset="VDDLEDS" device=""/>
 <part name="VDDLEDS5" library="BASTL_SYMBOLS" library_urn="urn:adsk.eagle:library:32975873" deviceset="VDDLEDS" device=""/>
-<part name="SW2" library="BASTL_SWITCHES" library_urn="urn:adsk.eagle:library:32903743" deviceset="EVQ-P7J01P" device="" package3d_urn="urn:adsk.eagle:package:45099218/2"/>
+<part name="SW2" library="BASTL_SWITCHES" library_urn="urn:adsk.eagle:library:32903743" deviceset="EVQ-P7J01P" device="" package3d_urn="urn:adsk.eagle:package:45099218/2" value="TSC4A 160gf-WZ 016"/>
 <part name="GND14" library="BASTL_SYMBOLS" library_urn="urn:adsk.eagle:library:32975873" deviceset="GND" device=""/>
 <part name="C9" library="BASTL_CAPACITORS" library_urn="urn:adsk.eagle:library:32978038" deviceset="CAPACITOR0603" device="" package3d_urn="urn:adsk.eagle:package:32978072/2" value="1u"/>
@@
 <part name="GND22" library="BASTL_SYMBOLS" library_urn="urn:adsk.eagle:library:32975873" deviceset="GND" device=""/>
 <part name="SJ1" library="BASTL_JUMPERS" library_urn="urn:adsk.eagle:library:32977727" deviceset="SMALL_NC" device="" package3d_urn="urn:adsk.eagle:package:45902385/1"/>
-<part name="Q2" library="BASTL_TRANZISTORS" library_urn="urn:adsk.eagle:library:32975847" deviceset="N-MOSFET" device="" package3d_urn="urn:adsk.eagle:package:32975863/4"/>
+<part name="Q2" library="BASTL_TRANZISTORS" library_urn="urn:adsk.eagle:library:32975847" deviceset="N-MOSFET" device="" package3d_urn="urn:adsk.eagle:package:32975863/4" value="2302"/>
 <part name="D2" library="BASTL_DIODES" library_urn="urn:adsk.eagle:library:32977972" deviceset="SCHOTTKY_DIODE" device="_SOD523" package3d_urn="urn:adsk.eagle:package:42502794/4" value="RB521S"/>
 <part name="D3" library="BASTL_DIODES" library_urn="urn:adsk.eagle:library:32977972" deviceset="SCHOTTKY_DIODE" device="_SOD523" package3d_urn="urn:adsk.eagle:package:42502794/4" value="RB521S"/>
@@
 <plain>
 <text x="24.384" y="-19.05" size="1.27" layer="94" ratio="12">Just for layout.</text>
-<text x="231.14" y="106.68" size="3.048" layer="98">REWORK THIS SECTION:
-REPLACE VBUS_FUSED
-WITH VSEL</text>
 <text x="-39.116" y="-34.29" size="1.27" layer="94" ratio="12">Just for layout.</text>
 </plain>
@@
 </instance>
 <instance part="F1" gate="G$1" x="-127" y="66.04" smashed="yes">
-<attribute name="NAME" x="-127" y="69.723" size="1.778" layer="95" align="center"/>
-<attribute name="VALUE" x="-127.127" y="62.23" size="1.778" layer="96" align="center"/>
+<attribute name="NAME" x="-127" y="72.263" size="1.778" layer="95" align="center"/>
+<attribute name="VALUE" x="-122.047" y="69.85" size="1.778" layer="96" align="center"/>
 </instance>
 <instance part="GND1" gate="1" x="-167.64" y="40.64" smashed="yes">
@@
 </drawing>
 <compatibility>
-<note version="6.3" minversion="6.2.2" severity="warning">
-Since Version 6.2.2 text objects can contain more than one line,
-which will not be processed correctly with this version.
-</note>
 <note version="8.2" severity="warning">
 Since Version 8.2, EAGLE supports online libraries. The ids
