File: pcb/sw63_mk4_v1/sw63_mk4_v1.kicad_pcb (KiCad board)
At the start: 2 copper layers, 81.3 x 48.3 mm, 51 parts, among them J1 Conn_01x08_Pin, J2 Conn_01x08_Pin, J3 Conn_01x03_Pin, J4 Conn_01x03_Pin, J5 Conn_01x03_Pin, J6 Conn_01x03_Pin, Q1 Q_PMOS_GSD, Q2 Q_PMOS_GSD, Q3 Q_PMOS_GSD, Q4 Q_PMOS_GSD, SW1 SW_Push, U1 TLC5916, U2 TLC5916, U3 TLC5916, U4 DS3231MZ

Commit message: layout in progress
Parts:
- removed J3, J4, J5, J6: Conn_01x03_Pin, Connector_PinHeader_2.54mm:PinHeader_1x03_P2.54mm_Vertical
- removed JP1: SolderJumper_3_Open, Jumper:SolderJumper-3_P2.0mm_Open_TrianglePad1.0x1.5mm
- removed Q4: Q_PMOS_GSD, Package_TO_SOT_SMD:SOT-23
- added C10: 100n, Capacitor_SMD:C_0402_1005Metric, B.Cu at (184.8, 128.4)
- added C11: 100n, Capacitor_SMD:C_0402_1005Metric, B.Cu at (184.8, 130.4)
- added C12: 100n, Capacitor_SMD:C_0402_1005Metric, B.Cu at (184.8, 132.4)
- added C6: 100n, Capacitor_SMD:C_0402_1005Metric, B.Cu at (184.8, 120.5)
- added C7: 10u, Capacitor_SMD:C_0402_1005Metric, B.Cu at (184.8, 122.5)
- added C8: 10u, Capacitor_SMD:C_0402_1005Metric, B.Cu at (184.8, 124.5)
- added C9: 100n, Capacitor_SMD:C_0402_1005Metric, B.Cu at (184.8, 126.5)
- added D22: MS2A40LWS, Diode_SMD:D_SOD-323, B.Cu at (197.5, 121.0)
- added F1: 0603L020/30XR, Fuse:Fuse_0603_1608Metric, B.Cu at (197.3, 123.8)
- added R10: 4k7, Resistor_SMD:R_0402_1005Metric, B.Cu at (190.6, 129.1)
- added R11: 100k, Resistor_SMD:R_0402_1005Metric, B.Cu at (190.6, 131.1)
- added R12: 100k, Resistor_SMD:R_0402_1005Metric, B.Cu at (193.5, 127.1)
- added R13: 220k, Resistor_SMD:R_0402_1005Metric, B.Cu at (193.5, 129.1)
- added R14: 22k, Resistor_SMD:R_0402_1005Metric, B.Cu at (193.5, 131.1)
- added R6: 10k, Resistor_SMD:R_0402_1005Metric, B.Cu at (187.7, 127.1)
- added R7: 10k, Resistor_SMD:R_0402_1005Metric, B.Cu at (187.7, 129.1)
- added R8: 2k, Resistor_SMD:R_0402_1005Metric, B.Cu at (187.7, 131.1)
- added R9: 4k7, Resistor_SMD:R_0402_1005Metric, B.Cu at (190.6, 127.1)
- added SW2: ﻿EVQ-P7J01P, Button_Switch_SMD:SW_SPST_EVQP7A, B.Cu at (198.2, 135.7)
- added U5: TLC5916, Package_SO:TSSOP-16_4.4x5mm_P0.65mm, B.Cu at (208.9, 84.9)
- added U6: DS3231MZ, Package_SO:SOIC-8_3.9x4.9mm_P1.27mm, B.Cu at (190.4, 135.5)
- added U7: STM32L052K8Ux, Package_DFN_QFN:QFN-32-1EP_5x5mm_P0.5mm_EP3.45x3.45mm, B.Cu at (199.0, 129.8)
- C1, C2, C3: value 100n -> 10u; footprint Capacitor_SMD:C_0603_1608Metric_Pad1.08x0.95mm_HandSolder -> Capacitor_SMD:C_0402_1005Metric; moved to B.Cu
- C4, C5: footprint Capacitor_SMD:C_0603_1608Metric_Pad1.08x0.95mm_HandSolder -> Capacitor_SMD:C_0402_1005Metric; moved to B.Cu
- H1, H2, H3, H4: footprint MountingHole:MountingHole_3.2mm_M3_DIN965 -> sw63_mk4:MountingHole_1.6mm
- J1: value Conn_01x08_Pin -> USB_C_Receptacle_USB2.0_16P; footprint Connector_PinHeader_2.54mm:PinHeader_1x08_P2.54mm_Vertical -> Connector_USB:USB_C_Receptacle_XKB_U262-16XN-4BVC11
- J2: value Conn_01x08_Pin -> Conn_ARM_JTAG_SWD_10; footprint Connector_PinHeader_2.54mm:PinHeader_1x08_P2.54mm_Vertical -> Connector_PinHeader_1.27mm:PinHeader_2x05_P1.27mm_Vertical_SMD
- Q1: value Q_PMOS_GSD -> DMG2305UX-7; moved to B.Cu
- Q2: value Q_PMOS_GSD -> DMG2302U-7; moved to B.Cu
- Q3: value Q_PMOS_GSD -> TEMT6200FX01; footprint Package_TO_SOT_SMD:SOT-23 -> Diode_SMD:D_0805_2012Metric; moved to B.Cu
- R1, R2: value 10k -> 5k1; footprint Resistor_SMD:R_0603_1608Metric_Pad0.98x0.95mm_HandSolder -> Resistor_SMD:R_0402_1005Metric; moved to B.Cu
- R3: value 2k -> 22k; footprint Resistor_SMD:R_0603_1608Metric_Pad0.98x0.95mm_HandSolder -> Resistor_SMD:R_0402_1005Metric; moved to B.Cu
- R4, R5: value 4k7 -> 10k; footprint Resistor_SMD:R_0603_1608Metric_Pad0.98x0.95mm_HandSolder -> Resistor_SMD:R_0402_1005Metric; moved to B.Cu
- SW1: value SW_Push -> KSC321J LFS; footprint Button_Switch_THT:SW_PUSH_6mm -> Button_Switch_SMD:SW_Push_1P1T_NO_CK_KSC6xxJ
- U1: value TLC5916 -> DIO5518BST5; footprint Package_SO:TSSOP-16_4.4x5mm_P0.65mm -> Package_TO_SOT_SMD:SOT-23-5; moved to B.Cu
- U2: value TLC5916 -> MCP1711T-3.3I/OT; footprint Package_SO:TSSOP-16_4.4x5mm_P0.65mm -> Package_TO_SOT_SMD:SOT-23-5; moved to B.Cu
- U3: moved to B.Cu
- U4: value DS3231MZ -> TLC5916; footprint Package_SO:SOIC-8_3.9x4.9mm_P1.27mm -> Package_SO:TSSOP-16_4.4x5mm_P0.65mm; moved to B.Cu
- moved D13 122.6 mm to (209.0, 60.5)
- moved D1 111.5 mm to (195.5, 68.0)
- moved D12 109.8 mm to (221.5, 67.0)
- moved D11 109.3 mm to (218.5, 67.0)
- moved D10 109.3 mm to (216.0, 67.5)
- moved D14 108.5 mm to (202.5, 61.0)
- moved D9 108.3 mm to (212.5, 67.5)
- moved D8 107.9 mm to (209.5, 67.5)
- moved D7 106.9 mm to (206.0, 67.5)
- moved D6 106.4 mm to (203.0, 68.0)
- moved D5 105.9 mm to (200.0, 68.0)
- moved D2 105.2 mm to (191.6, 68.2)
- moved H1 102.3 mm to (181.6, 53.1)
- moved R1 102.3 mm to (185.8, 75.8)
- moved C4 102.3 mm to (237.4, 80.7), turned to 0 degrees
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Connections:
- C1 pad 1: VDD -> VBUS
- C2 pad 1: VDD -> VBUS
- C3 pad 1: VDD -> /VBAT
- C4 pad 1: /RTC_VBAT -> /VSEL
- C4 pad 2: /RTC_GND -> GND
- C5 pad 1: /RTC_VCC -> /VSEL
- C5 pad 2: /RTC_GND -> GND
- D1 pad 2: VDD -> /VSEL
- D10 pad 2: VDD -> /VSEL
- D11 pad 2: VDD -> /VSEL
- D12 pad 2: VDD -> /VSEL
- D13 pad 2: VDD -> /VSEL
- D14 pad 2: VDD -> /VSEL
- D15 pad 2: VDD -> /VSEL
- D16 pad 2: VDD -> /VSEL
- D17 pad 2: VDD -> /VSEL
- D18 pad 2: VDD -> /VSEL
- D19 pad 2: VDD -> /VSEL
- D2 pad 2: VDD -> /VSEL
- D20 pad 2: VDD -> /VSEL
- D21 pad 2: VDD -> /VSEL
- D3 pad 2: VDD -> /VSEL
- D4 pad 2: VDD -> /VSEL
- D5 pad 2: VDD -> /VSEL
- D6 pad 2: VDD -> /VSEL
- D7 pad 2: VDD -> /VSEL
- D8 pad 2: VDD -> /VSEL
- D9 pad 2: VDD -> /VSEL
- J2 pad 1: /RTC_GND -> VDD
- J2 pad 2: /RTC_VCC -> /SWDIO
- J2 pad 3: /RTC_VBAT -> GND
- J2 pad 4: /SDA -> /SWCLK
- J2 pad 5: /SCL -> GND
- J2 pad 6: /!RST -> unconnected-(J2-SWO/TDO-Pad6)
- J2 pad 7: /!INT -> unconnected-(J2-KEY-Pad7)
- J2 pad 8: /32KHZ -> unconnected-(J2-NC/TDI-Pad8)
- Q1 pad 1: Net-(J3-Pin_1) -> VBUS
- Q1 pad 2: Net-(J3-Pin_2) -> /VSEL
- Q1 pad 3: Net-(J3-Pin_3) -> /VBAT
- Q2 pad 1: Net-(J4-Pin_1) -> /ACTIVE
- Q2 pad 3: Net-(J4-Pin_3) -> GND
- Q3 pad 1: Net-(J5-Pin_1) -> /ACTIVE
- Q3 pad 2: Net-(J5-Pin_2) -> /AMBIENT_LIGHT
- R1 pad 1: Net-(U1-R-EXT) -> Net-(J1-CC1)
- R2 pad 1: Net-(U2-R-EXT) -> Net-(J1-CC2)
- R3 pad 1: Net-(U3-R-EXT) -> Net-(U1-PROG)
- R4 pad 1: Net-(JP1-C) -> VBUS
- R4 pad 2: /SDA -> GND
- R5 pad 1: Net-(JP1-C) -> VDD
- R5 pad 2: /SCL -> /!RESET
- SW1 pad 1: /BTN_B -> GND
- SW1 pad 2: /BTN_A -> /BTN
- U1 pad 1: GND -> /CHRG_STAT
- U1 pad 2: /DATA -> GND
- U1 pad 3: /CLOCK -> /VBAT
- U1 pad 4: /LATCH -> VBUS
- U1 pad 5: Net-(D5-K) -> Net-(U1-PROG)
- U2 pad 1: GND -> /VSEL
- U2 pad 2: Net-(U1-SDO) -> GND
- U2 pad 3: /CLOCK -> /VSEL
- U2 pad 4: /LATCH -> unconnected-(U2-NC-Pad4)
- U2 pad 5: Net-(D9-K) -> VDD
- U3 pad 10: Net-(D18-K) -> Net-(D6-K)
- U3 pad 11: Net-(D19-K) -> Net-(D7-K)
- U3 pad 12: Net-(D20-K) -> Net-(D8-K)
- U3 pad 14: unconnected-(U3-SDO-Pad14) -> Net-(U3-SDO)
- U3 pad 2: Net-(U2-SDO) -> /DATA
- U3 pad 5: unconnected-(U3-~{OUT0}-Pad5) -> Net-(D1-K)
- U3 pad 6: unconnected-(U3-~{OUT1}-Pad6) -> Net-(D2-K)
- U3 pad 7: unconnected-(U3-~{OUT2}-Pad7) -> Net-(D3-K)
- U3 pad 8: Net-(D21-K) -> Net-(D4-K)
- U3 pad 9: Net-(D17-K) -> Net-(D5-K)
- U4 pad 1: /32KHZ -> GND
- U4 pad 2: /RTC_VCC -> Net-(U3-SDO)
- U4 pad 3: /!INT -> /CLOCK
- U4 pad 4: /!RST -> /LATCH
- U4 pad 5: /RTC_GND -> Net-(D9-K)
- U4 pad 6: /RTC_VBAT -> Net-(D10-K)
- U4 pad 7: /SDA -> Net-(D11-K)
- U4 pad 8: /SCL -> Net-(D12-K)
Routing:
- net VDD: track 178.5 -> 0.00 mm, vias 3 -> 0
- net /RTC_VCC: track 59.9 -> 0.00 mm
- net /LATCH: track 56.0 -> 0.00 mm, vias 5 -> 0
- net /!OE: track 54.2 -> 0.00 mm, vias 6 -> 0
- net /CLOCK: track 44.7 -> 0.00 mm
- net Net-(D17-K): track 40.0 -> 0.00 mm
- net /RTC_VBAT: track 36.9 -> 0.00 mm, vias 2 -> 0
- net /!RST: track 27.6 -> 0.00 mm
- net /!INT: track 26.6 -> 0.00 mm
- net Net-(D18-K): track 26.4 -> 0.00 mm
- net /32KHZ: track 26.4 -> 0.00 mm
- net Net-(D13-K): track 24.4 -> 0.00 mm, vias 1 -> 0
- net Net-(D8-K): track 24.2 -> 0.00 mm
- net /SDA: track 23.3 -> 0.00 mm
- net /BTN_B: track 22.1 -> 0.00 mm
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- removed copper zone on B.Cu, net /RTC_GND
- removed copper zone on F.Cu, net /RTC_GND
- removed copper zone on B.Cu, net GND
- removed copper zone on F.Cu, net GND
Other:
- board outline removed
- board text added: "SW63 Mk4"
- board text removed: "32kHz"
- board text removed: "BTN_A"
- board text removed: "BTN_B"
- board text removed: "BUTTON"
- board text removed: "CLOCK"
- board text removed: "D"
- board text removed: "DATA"
- board text removed: "DISPLAY"
- board text removed: "G"
- board text removed: "GND"
- board text removed: "I2C pull-ups"
- board text removed: "LATCH"
- board text removed: "RTC"
- board text removed: "S"
- board text removed: "SCL"
- board text removed: "SDA"
- board text removed: "SW63 Mk4 dev board"
- board text removed: "UTILS"
- board text removed: "VBAT"
- board text removed: "VCC"
- board text removed: "VDD"
- board text removed: "~{INT}"
- board text removed: "~{OE}"
- board text removed: "~{RST}"

Commit message: update board
Parts:
- J1: footprint Connector_USB:USB_C_Receptacle_XKB_U262-16XN-4BVC11 -> sw63_mk4:GT-USB-7070C
- SW1: footprint Button_Switch_SMD:SW_Push_1P1T_NO_CK_KSC6xxJ -> sw63_mk4:SW_Push_1P1T_NO_CK_KSC3xxJ
- turned J1 to 90 degrees

Commit message: update board
Parts:
- added J3: Conn_01x02, sw63_mk4:BAT, B.Cu at (105.8, 77.7)
- J2: value Conn_ARM_JTAG_SWD_10 -> SWD; footprint Connector_PinHeader_1.27mm:PinHeader_2x05_P1.27mm_Vertical_SMD -> sw63_mk4:SWD_2x03_SMD
- Q3: moved to F.Cu
- moved C4 139.9 mm to (97.6, 75.0), turned to -90 degrees
- moved C5 138.3 mm to (101.1, 71.0), turned to -90 degrees
- moved Q3 131.2 mm to (121.6, 86.6), turned to 0 degrees
- moved Q2 129.0 mm to (113.9, 87.3), turned to 0 degrees
- moved H3 127.0 mm to (131.5, 75.0)
- moved H2 125.2 mm to (131.5, 90.0)
- moved J2 111.8 mm to (115.0, 95.5)
- moved Q1 111.7 mm to (127.0, 71.3)
- moved R5 107.6 mm to (131.5, 100.5)
- moved U7 98.9 mm to (112.5, 81.7), turned to 90 degrees
- moved U6 98.2 mm to (117.5, 69.7), turned to -90 degrees
- moved C6 96.9 mm to (96.4, 80.8)
- moved D12 90.6 mm to (132.2, 82.5)
- moved D10 90.4 mm to (126.9, 82.5)
- moved D11 90.3 mm to (129.5, 82.5)
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Connections:
- C4 pad 2: GND -> /GND_LED
- C5 pad 2: GND -> /GND_LED
- C6 pad 2: GND -> /GND_LED
- J2 pad 3: GND -> /!RESET
- Q2 pad 2: Net-(Q2-D) -> /GND_LED
- R6 pad 2: Net-(Q2-D) -> /GND_LED
- R7 pad 2: Net-(Q2-D) -> /GND_LED
- R8 pad 2: Net-(Q2-D) -> /GND_LED
- U3 pad 1: GND -> /GND_LED
- U3 pad 16: VDD -> /VSEL
- U4 pad 1: GND -> /GND_LED
- U4 pad 10: Net-(D14-K) -> Net-(D15-K)
- U4 pad 11: Net-(D15-K) -> Net-(D14-K)
- U4 pad 12: Net-(D16-K) -> Net-(D13-K)
- U4 pad 16: VDD -> /VSEL
- U4 pad 9: Net-(D13-K) -> Net-(D16-K)
- U5 pad 1: GND -> /GND_LED
- U5 pad 16: VDD -> /VSEL
Other:
- board outline added: 35 x 35 mm

Commit message: update models and footprints
Parts:
- D1, D10, D11, D12, D2, D3, D4, D5, D6, D7, D8, D9: footprint LED_SMD:LED_1206_3216Metric_Pad1.42x1.75mm_HandSolder -> sw63_mk4:LED_1206_W
- D13: footprint LED_THT:LED_D5.0mm -> sw63_mk4:LED_D5.0mm_Y
- D14: footprint LED_THT:LED_D5.0mm -> sw63_mk4:LED_D5.0mm_B
- D15: footprint LED_THT:LED_D5.0mm -> sw63_mk4:LED_D5.0mm_G
- D16: footprint LED_THT:LED_D5.0mm -> sw63_mk4:LED_D5.0mm_R
- D17, D18, D19, D20: footprint LED_THT:LED_D2.0mm_W4.0mm_H2.8mm_FlatTop -> sw63_mk4:LED_W3.0mm_H2.0mm_Y
- D21: footprint LED_THT:LED_D3.0mm -> sw63_mk4:LED_D3.0mm_R
- moved D21 0.16 mm to (129.1, 89.6)

Commit message: routing in progress
Parts:
- moved R13 61.5 mm to (103.2, 77.5), turned to 0 degrees
- moved R11 59.9 mm to (103.2, 78.7)
- moved R10 51.9 mm to (114.2, 77.2), turned to 0 degrees
- moved C12 51.6 mm to (117.5, 75.0), turned to -90 degrees
- moved R9 49.1 mm to (116.3, 77.2)
- moved C9 48.2 mm to (110.2, 77.9)
- moved R6 48.2 mm to (108.2, 83.3), turned to 90 degrees
- moved C7 47.7 mm to (121.8, 67.4), turned to 0 degrees
- moved C8 46.6 mm to (125.1, 69.2), turned to -90 degrees
- moved R7 45.8 mm to (120.5, 78.3), turned to 90 degrees
- moved R12 45.1 mm to (112.8, 89.7), turned to 0 degrees
- moved C10 44.0 mm to (109.9, 85.9)
- moved R14 42.4 mm to (123.8, 86.1), turned to 90 degrees
- moved C11 42.2 mm to (114.8, 85.8), turned to 0 degrees
- moved R8 40.8 mm to (115.5, 90.4), turned to -90 degrees
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Connections:
- U5 pad 10: Net-(D18-K) -> Net-(D20-K)
- U5 pad 11: Net-(D19-K) -> Net-(D17-K)
- U5 pad 12: Net-(D20-K) -> Net-(D18-K)
- U5 pad 9: Net-(D17-K) -> Net-(D19-K)
- U6 pad 1: /32KHZ -> unconnected-(U6-32KHZ-Pad1)
- U6 pad 3: /!INT -> unconnected-(U6-~{INT}/SQW-Pad3)
- U6 pad 4: /!RST -> unconnected-(U6-~{RST}-Pad4)
Routing:
- net /VSEL: track 0.00 -> 24.1 mm
- net /!RESET: track 0.00 -> 19.6 mm
- net /VBAT: track 0.00 -> 17.5 mm
- net Net-(D17-K): track 0.00 -> 17.3 mm
- net VDD: track 0.00 -> 13.8 mm
- net Net-(D20-K): track 0.00 -> 13.6 mm
- net VBUS: track 0.00 -> 11.9 mm
- net Net-(F1-Pad1): track 0.00 -> 11.8 mm
- net Net-(D19-K): track 0.00 -> 8.06 mm
- net Net-(D21-K): track 0.00 -> 7.88 mm
- net Net-(D18-K): track 0.00 -> 3.30 mm
- net Net-(U1-PROG): track 0.00 -> 2.00 mm
- net Net-(U4-R-EXT): track 0.00 -> 1.84 mm
- net GND: track 0.00 -> 1.59 mm
- net /BATTERY_LEVEL: track 0.00 -> 1.25 mm
Other:
- copper layers 2 -> 4

Commit message: routing
Parts:
- moved R12 3.37 mm to (112.2, 93.0)
- moved C10 2.97 mm to (112.8, 85.8), turned to 0 degrees
- moved Q2 1.41 mm to (112.7, 88.7), turned to -90 degrees
- moved C2 1.11 mm to (124.1, 78.7)
- moved R14 1.00 mm to (123.8, 87.1), turned to -90 degrees
- moved C4 0.61 mm to (107.7, 81.0)
- moved R6 0.61 mm to (107.7, 83.0), turned to -90 degrees
- moved C12 0.55 mm to (117.5, 74.5), turned to 90 degrees
- moved U3 0.48 mm to (104.3, 84.1)
- moved C11 0.38 mm to (115.2, 85.8)
- moved R13 0.10 mm to (103.2, 77.5)
Routing:
- net /VSEL: track 24.1 -> 134.9 mm, vias 0 -> 6
- net VDD: track 13.8 -> 78.9 mm, vias 0 -> 6
- net /!OE: track 0.00 -> 58.5 mm, vias 0 -> 5
- net /GND_LED: track 0.00 -> 57.5 mm, vias 0 -> 7
- net /LATCH: track 0.00 -> 54.8 mm, vias 0 -> 3
- net /CLOCK: track 0.00 -> 44.7 mm, vias 0 -> 2
- net Net-(U3-SDO): track 0.00 -> 39.0 mm, vias 0 -> 3
- net /VBAT: track 17.5 -> 46.6 mm, vias 0 -> 3
- net /SWDIO: track 0.00 -> 27.6 mm, vias 0 -> 3
- net /D-: track 0.00 -> 26.4 mm, vias 0 -> 3
- net /AMBIENT_LIGHT: track 0.00 -> 25.6 mm, vias 0 -> 2
- net /!RESET: track 19.6 -> 44.4 mm, vias 0 -> 2
- net /CHRG_STAT: track 0.00 -> 24.7 mm, vias 0 -> 3
- net /SWCLK: track 0.00 -> 24.7 mm, vias 0 -> 2
- net /D+: track 0.00 -> 24.5 mm, vias 0 -> 2
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Other:
- board text added: "RST"
- board text added: "space"
- board text added: "watch"
- board text added: "xx0x"

Commit message: routing
Parts:
- moved R2 0.43 mm to (124.1, 83.9)
- moved C11 0.40 mm to (115.2, 86.2)
- moved J3 0.12 mm to (107.5, 77.9)
- moved C2 0.05 mm to (124.1, 78.6)
Routing:
- net GND: track 1.59 -> 33.5 mm, vias 0 -> 25
- net /GND_LED: track 57.5 -> 62.7 mm, vias 7 -> 6
- net /VSEL: track 134.9 -> 137.8 mm
- net /DATA: track 9.88 -> 7.27 mm, vias 1 -> 0
- net /CHRG_STAT: track 24.7 -> 23.2 mm
- net Net-(U3-SDO): track 39.0 -> 40.4 mm
- net /CLOCK: track 44.7 -> 45.7 mm
- net VDD: track 78.9 -> 78.1 mm
- net /!RESET: track 44.4 -> 45.0 mm
- net /SWDIO: track 27.6 -> 28.1 mm
- added copper zone on B.Cu, net GND
- added copper zone on F.Cu, net GND
- added copper zone on In1.Cu, net GND
- added copper zone on In2.Cu, net GND
Other:
- board text added: "+"
- board text added: "-"
- board text added: "BAT"

Commit message: routing
Parts:
- moved Q2 0.11 mm to (112.7, 88.8)
Routing:
- net /AMBIENT_LIGHT: track 25.4 -> 21.0 mm
- net Net-(D1-K): track 12.7 -> 12.2 mm
