File: pcb/sw63_mk4_v1/sw63_mk4_v1.kicad_sch (KiCad schematic)
At the start: 67 parts, among them J7 USB_C_Receptacle_USB2.0_16P, J8 Conn_ARM_JTAG_SWD_10, Q1 DMG2302U-7, Q2 TEMT6200FX01, Q5 DMG2305UX-7, SW1 KSC321J LFS, SW2 ﻿EVQ-P7J01P, U1 TLC5916, U2 TLC5916, U3 TLC5916, U4 DS3231MZ, U5 STM32L052K8Ux, U6 MCP1711T-3.3I/OT, U7 DIO5518BST5

Commit message: layout in progress
Parts:
- C1: renamed from C11; footprint Capacitor_SMD:C_0805_2012Metric -> Capacitor_SMD:C_0402_1005Metric
- C10: renamed from C7; footprint Capacitor_SMD:C_0603_1608Metric -> Capacitor_SMD:C_0402_1005Metric
- C11, C9: renamed from C6; footprint Capacitor_SMD:C_0603_1608Metric -> Capacitor_SMD:C_0402_1005Metric
- C12: renamed from C4; footprint Capacitor_SMD:C_0603_1608Metric_Pad1.08x0.95mm_HandSolder -> Capacitor_SMD:C_0402_1005Metric
- C2: renamed from C7; footprint Capacitor_SMD:C_0805_2012Metric -> Capacitor_SMD:C_0402_1005Metric
- C3: renamed from C10; footprint Capacitor_SMD:C_0805_2012Metric -> Capacitor_SMD:C_0402_1005Metric
- C4: renamed from C1; footprint Capacitor_SMD:C_0603_1608Metric_Pad1.08x0.95mm_HandSolder -> Capacitor_SMD:C_0402_1005Metric
- C5: renamed from C2; footprint Capacitor_SMD:C_0603_1608Metric_Pad1.08x0.95mm_HandSolder -> Capacitor_SMD:C_0402_1005Metric
- C6: renamed from C3; footprint Capacitor_SMD:C_0603_1608Metric_Pad1.08x0.95mm_HandSolder -> Capacitor_SMD:C_0402_1005Metric
- C7: renamed from C9; footprint Capacitor_SMD:C_0805_2012Metric -> Capacitor_SMD:C_0402_1005Metric
- C8: footprint Capacitor_SMD:C_0805_2012Metric -> Capacitor_SMD:C_0402_1005Metric
- F1: value Polyfuse 200mA -> 0603L020/30XR; footprint Fuse:Fuse_0805_2012Metric -> Fuse:Fuse_0603_1608Metric; LCSC C883109 -> C20608677
- H1, H2, H3: footprint MountingHole:MountingHole_3.2mm_M3_DIN965 -> sw63_mk4:MountingHole_1.6mm
- Q2: renamed from Q1; footprint (none) -> Package_TO_SOT_SMD:SOT-23
- R1: renamed from R6; footprint Resistor_SMD:R_0603_1608Metric -> Resistor_SMD:R_0402_1005Metric
- R10: renamed from R5; footprint Resistor_SMD:R_0603_1608Metric_Pad0.98x0.95mm_HandSolder -> Resistor_SMD:R_0402_1005Metric
- R11: renamed from R13; footprint Resistor_SMD:R_0603_1608Metric -> Resistor_SMD:R_0402_1005Metric
- R12: renamed from R11; footprint Resistor_SMD:R_0603_1608Metric_Pad0.98x0.95mm_HandSolder -> Resistor_SMD:R_0402_1005Metric
- R13: renamed from R14; footprint Resistor_SMD:R_0603_1608Metric -> Resistor_SMD:R_0402_1005Metric
- R14: renamed from R12; footprint Resistor_SMD:R_0603_1608Metric_Pad0.98x0.95mm_HandSolder -> Resistor_SMD:R_0402_1005Metric
- R2, R5: renamed from R7; footprint Resistor_SMD:R_0603_1608Metric -> Resistor_SMD:R_0402_1005Metric
- R3: renamed from R10; footprint Resistor_SMD:R_0603_1608Metric -> Resistor_SMD:R_0402_1005Metric
- R4: renamed from R8; footprint Resistor_SMD:R_0603_1608Metric -> Resistor_SMD:R_0402_1005Metric
- R6: renamed from R1; footprint Resistor_SMD:R_0603_1608Metric_Pad0.98x0.95mm_HandSolder -> Resistor_SMD:R_0402_1005Metric
- R7: renamed from R2; footprint Resistor_SMD:R_0603_1608Metric_Pad0.98x0.95mm_HandSolder -> Resistor_SMD:R_0402_1005Metric
- R8: renamed from R3; footprint Resistor_SMD:R_0603_1608Metric_Pad0.98x0.95mm_HandSolder -> Resistor_SMD:R_0402_1005Metric
- R9: renamed from R4; footprint Resistor_SMD:R_0603_1608Metric_Pad0.98x0.95mm_HandSolder -> Resistor_SMD:R_0402_1005Metric
- renumbered J7 to J1, J8 to J2, Q5 to Q1, Q2 to Q3, U7 to U1, U6 to U2, U1 to U3, U2 to U4, U3 to U5, U4 to U6, U5 to U7
Connections:
- net at D7.1 (K): now also U3.11 (~{OUT6}); no longer U3.7 (~{OUT2})
- net at U3.10 (~{OUT5}): now also D6.1 (K); no longer D3.1 (K)
- net at D2.1 (K): now also U3.6 (~{OUT1}); no longer U3.11 (~{OUT6})
- net at U3.12 (~{OUT7}): now also D8.1 (K); no longer D1.1 (K)
- net at U3.5 (~{OUT0}): now also D1.1 (K); no longer D5.1 (K)
- net at U3.8 (~{OUT3}): now also D4.1 (K); no longer D8.1 (K)
- net at U3.9 (~{OUT4}): now also D5.1 (K); no longer D4.1 (K)
- net at U4.10 (~{OUT5}): now also D14.1 (K); no longer D15.1 (K)
- net at U4.11 (~{OUT6}): now also D15.1 (K); no longer D14.1 (K)
- net at U4.12 (~{OUT7}): now also D16.1 (K); no longer D13.1 (K)
- net at U4.9 (~{OUT4}): now also D13.1 (K); no longer D16.1 (K)
- new net: D3.1 (K), U3.7 (~{OUT2})
Other:
- moved on the sheet: C7, C8, D1, D10, D11, D12, D13, D14, D15, D16, D17, D18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

Commit message: update board
Parts:
- J1: footprint Connector_USB:USB_C_Receptacle_XKB_U262-16XN-4BVC11 -> sw63_mk4:GT-USB-7070C; LCSC C393939 -> C5446864
- SW1: footprint Button_Switch_SMD:SW_Push_1P1T_NO_CK_KSC6xxJ -> sw63_mk4:SW_Push_1P1T_NO_CK_KSC3xxJ
Changed lines of the file:
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@@
 			)
 		)
-		(property "Footprint" "Button_Switch_SMD:SW_Push_1P1T_NO_CK_KSC6xxJ"
+		(property "Footprint" "sw63_mk4:SW_Push_1P1T_NO_CK_KSC3xxJ"
 			(at 77.47 88.9 0)
 			(effects
@@
 			)
 		)
-		(property "Footprint" "Connector_USB:USB_C_Receptacle_XKB_U262-16XN-4BVC11"
+		(property "Footprint" "sw63_mk4:GT-USB-7070C"
 			(at 36.83 48.26 0)
 			(effects
@@
 			)
 		)
-		(property "LCSC" "C393939"
+		(property "LCSC" "C5446864"
 			(at 33.02 25.4 0)
 			(effects
@@
 			)
 		)
-		(property "Description" "Ambient Light Sensor"
+		(property "Description" "NPN phototransistor, collector/emitter"
 			(at 157.48 176.53 0)
 			(effects

Commit message: update board
Parts:
- removed J2: Conn_ARM_JTAG_SWD_10, Connector_PinHeader_1.27mm:PinHeader_2x05_P1.27mm_Vertical_SMD, symbol Connector:Conn_ARM_JTAG_SWD_10
- added J2: SWD, sw63_mk4:SWD_2x03_SMD, symbol Connector:Conn_ARM_SWD_TagConnect_TC2030
- added J3: Conn_01x02, sw63_mk4:BAT, symbol Connector_Generic:Conn_01x02
Connections:
- net !RESET: now also J2.3 (~{RESET})
- net GND: now also J2.5 (GND), J3.1 (Pin_1); no longer C4.2, C5.2, C6.2, U3.1 (GND), U4.1 (GND), U5.1 (GND)
- net SWCLK: now also J2.4 (SWCLK)
- net SWDIO: now also J2.2 (SWDIO)
- net VBAT: now also J3.2 (Pin_2)
- net VDD: now also J2.1 (VCC); no longer U3.16 (VDD), U4.16 (VDD), U5.16 (VDD)
- net VSEL: now also U3.16 (VDD), U4.16 (VDD), U5.16 (VDD)
- net GND_LED: now reaches Q2.2 (D), R6.2, R7.2, R8.2
- net GND_LED: now also C4.2, C5.2, C6.2, U3.1 (GND), U4.1 (GND), U5.1 (GND)
- net at U4.10 (~{OUT5}): now also D15.1 (K); no longer D14.1 (K)
- net at U4.11 (~{OUT6}): now also D14.1 (K); no longer D15.1 (K)
- net at U4.12 (~{OUT7}): now also D13.1 (K); no longer D16.1 (K)
- net at U4.9 (~{OUT4}): now also D16.1 (K); no longer D13.1 (K)
Other:
- moved on the sheet: C4, C5, C6, D13, D14, D15, D16

Commit message: update models and footprints
Parts:
- D1, D10, D11, D12, D2, D3, D4, D5, D6, D7, D8, D9: footprint LED_SMD:LED_1206_3216Metric_Pad1.42x1.75mm_HandSolder -> sw63_mk4:LED_1206_W
- D13: footprint LED_THT:LED_D5.0mm -> sw63_mk4:LED_D5.0mm_Y
- D14: footprint LED_THT:LED_D5.0mm -> sw63_mk4:LED_D5.0mm_B
- D15: footprint LED_THT:LED_D5.0mm -> sw63_mk4:LED_D5.0mm_G
- D16: footprint LED_THT:LED_D5.0mm -> sw63_mk4:LED_D5.0mm_R
- D17, D18, D19, D20: footprint LED_THT:LED_D2.0mm_W4.0mm_H2.8mm_FlatTop -> sw63_mk4:LED_W3.0mm_H2.0mm_Y
- D21: footprint LED_THT:LED_D3.0mm -> sw63_mk4:LED_D3.0mm_R
Changed lines of the file:
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@@
 			)
 		)
-		(property "Footprint" "LED_SMD:LED_1206_3216Metric_Pad1.42x1.75mm_HandSolder"
+		(property "Footprint" "sw63_mk4:LED_1206_W"
 			(at 168.91 81.28 0)
 			(effects
@@
 			)
 		)
-		(property "Footprint" "LED_THT:LED_D2.0mm_W4.0mm_H2.8mm_FlatTop"
+		(property "Footprint" "sw63_mk4:LED_W3.0mm_H2.0mm_Y"
 			(at 264.16 81.28 0)
 			(effects
@@
 			)
 		)
-		(property "Footprint" "LED_SMD:LED_1206_3216Metric_Pad1.42x1.75mm_HandSolder"
+		(property "Footprint" "sw63_mk4:LED_1206_W"
 			(at 158.75 81.28 0)
 			(effects
@@
 			)
 		)
-		(property "Footprint" "LED_THT:LED_D2.0mm_W4.0mm_H2.8mm_FlatTop"
+		(property "Footprint" "sw63_mk4:LED_W3.0mm_H2.0mm_Y"
 			(at 256.54 81.28 0)
 			(effects
@@
 			)
 		)
-		(property "Footprint" "LED_SMD:LED_1206_3216Metric_Pad1.42x1.75mm_HandSolder"
+		(property "Footprint" "sw63_mk4:LED_1206_W"
 			(at 153.67 81.28 0)
 			(effects
@@
 			)
 		)
-		(property "Footprint" "LED_SMD:LED_1206_3216Metric_Pad1.42x1.75mm_HandSolder"
+		(property "Footprint" "sw63_mk4:LED_1206_W"
 			(at 203.2 81.28 0)
 			(effects
@@
 			)
 		)
-		(property "Footprint" "LED_SMD:LED_1206_3216Metric_Pad1.42x1.75mm_HandSolder"
+		(property "Footprint" "sw63_mk4:LED_1206_W"
 			(at 163.83 81.28 0)
 			(effects
@@
 			)
 		)
-		(property "Footprint" "LED_SMD:LED_1206_3216Metric_Pad1.42x1.75mm_HandSolder"
+		(property "Footprint" "sw63_mk4:LED_1206_W"
 			(at 200.66 81.28 0)
 			(effects
@@
 			)
 		)
-		(property "Footprint" "LED_THT:LED_D2.0mm_W4.0mm_H2.8mm_FlatTop"
+		(property "Footprint" "sw63_mk4:LED_W3.0mm_H2.0mm_Y"
 			(at 261.62 81.28 0)
 			(effects
@@
 			)
 		)
-		(property "Footprint" "LED_THT:LED_D2.0mm_W4.0mm_H2.8mm_FlatTop"
+		(property "Footprint" "sw63_mk4:LED_W3.0mm_H2.0mm_Y"
 			(at 259.08 81.28 0)
 			(effects
@@
 			)
 		)
-		(property "Footprint" "LED_THT:LED_D5.0mm"
+		(property "Footprint" "sw63_mk4:LED_D5.0mm_B"
 			(at 215.9 81.28 0)
 			(effects
@@
 			)
 		)
-		(property "Footprint" "LED_SMD:LED_1206_3216Metric_Pad1.42x1.75mm_HandSolder"
+		(property "Footprint" "sw63_mk4:LED_1206_W"
 			(at 166.37 81.28 0)
 			(effects
@@
 			)
 		)
-		(property "Footprint" "LED_THT:LED_D5.0mm"
+		(property "Footprint" "sw63_mk4:LED_D5.0mm_Y"
 			(at 218.44 81.28 0)
 			(effects
@@
 			)
 		)
-		(property "Footprint" "LED_SMD:LED_1206_3216Metric_Pad1.42x1.75mm_HandSolder"
+		(property "Footprint" "sw63_mk4:LED_1206_W"
 			(at 171.45 81.28 0)
 			(effects
@@
 			)
 		)
-		(property "Footprint" "LED_SMD:LED_1206_3216Metric_Pad1.42x1.75mm_HandSolder"
+		(property "Footprint" "sw63_mk4:LED_1206_W"
 			(at 156.21 81.28 0)
 			(effects
@@
 			)
 		)
-		(property "Footprint" "LED_SMD:LED_1206_3216Metric_Pad1.42x1.75mm_HandSolder"
+		(property "Footprint" "sw63_mk4:LED_1206_W"
 			(at 161.29 81.28 0)
 			(effects
@@
 			)
 		)
-		(property "Footprint" "LED_THT:LED_D5.0mm"
+		(property "Footprint" "sw63_mk4:LED_D5.0mm_R"
 			(at 210.82 81.28 0)
 			(effects
@@
 			)
 		)
-		(property "Footprint" "LED_THT:LED_D3.0mm"
+		(property "Footprint" "sw63_mk4:LED_D3.0mm_R"
 			(at 254 81.28 0)
 			(effects
@@
 			)
 		)
-		(property "Footprint" "LED_SMD:LED_1206_3216Metric_Pad1.42x1.75mm_HandSolder"
+		(property "Footprint" "sw63_mk4:LED_1206_W"
 			(at 208.28 81.28 0)
 			(effects
@@
 			)
 		)
-		(property "Footprint" "LED_THT:LED_D5.0mm"
+		(property "Footprint" "sw63_mk4:LED_D5.0mm_G"
 			(at 213.36 81.28 0)
 			(effects
@@
 			)
 		)
-		(property "Footprint" "LED_SMD:LED_1206_3216Metric_Pad1.42x1.75mm_HandSolder"
+		(property "Footprint" "sw63_mk4:LED_1206_W"
 			(at 205.74 81.28 0)
 			(effects

Commit message: routing in progress
Connections:
- net at D20.1 (K): now also U5.10 (~{OUT5}); no longer U5.12 (~{OUT7})
- net at D17.1 (K): now also U5.11 (~{OUT6}); no longer U5.9 (~{OUT4})
- net at D19.1 (K): now also U5.9 (~{OUT4}); no longer U5.11 (~{OUT6})
- net at D18.1 (K): now also U5.12 (~{OUT7}); no longer U5.10 (~{OUT5})
- net !INT: no longer names the net of U6.3 (~{INT}/SQW)
- net !RST: no longer names the net of U6.4 (~{RST})
- net 32KHZ: no longer names the net of U6.1 (32KHZ)
Other:
- company: (none) -> github.com/xx0x/sw63
- title: (none) -> SW63 mk4
- moved on the sheet: C1, C10, C11, C12, C3, C4, C5, C6, C7, C8, C9, D17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

Commit message: routing, graphics
Parts:
- J1: value USB_C_Receptacle_USB2.0_16P -> GT-USB-7070C
- U3, U4, U5: value TLC5916 -> TLC5916IPWR
Other:
- note added: "BAT current when MCU sleeps (BAT is 4V) MCP73832T-2ACI/OT: approx 21uA - little worse DIO5518BST5: approx 15uA (10-20 based on ambient temperature) - little better"
- note removed: "BAT current when MCU sleeps (BAT is 4V) MCP73832T: approx 21uA - little worse DIO5518BST5: approx 15uA (10-20 based on ambient temperature) - little better"
Changed lines of the file:
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@@
 		(comment 3 "SW63")
 	)
-	(text "BAT current when MCU sleeps (BAT is 4V)\nMCP73832T: approx 21uA - little worse\nDIO5518BST5: approx 15uA (10-20 based on ambient temperature) - little better"
+	(text "BAT current when MCU sleeps (BAT is 4V)\nMCP73832T-2ACI/OT: approx 21uA - little worse\nDIO5518BST5: approx 15uA (10-20 based on ambient temperature) - little better"
 		(exclude_from_sim no)
 		(at 235.712 24.638 0)
@@
 		(fields_autoplaced yes)
 		(property "Reference" "U3"
-			(at 184.15 97.4246 90)
+			(at 186.69 97.4246 90)
 			(effects
 				(font
@@
 			)
 		)
-		(property "Value" "TLC5916"
-			(at 184.15 99.9646 90)
+		(property "Value" "TLC5916IPWR"
+			(at 186.69 99.9646 90)
 			(effects
 				(font
@@
 		(fields_autoplaced yes)
 		(property "Reference" "U4"
-			(at 231.14 97.4246 90)
+			(at 233.68 97.4246 90)
 			(effects
 				(font
@@
 			)
 		)
-		(property "Value" "TLC5916"
-			(at 231.14 99.9646 90)
+		(property "Value" "TLC5916IPWR"
+			(at 233.68 99.9646 90)
 			(effects
 				(font
@@
 		(fields_autoplaced yes)
 		(property "Reference" "U5"
-			(at 276.86 97.4246 90)
+			(at 279.4 97.4246 90)
 			(effects
 				(font
@@
 			)
 		)
-		(property "Value" "TLC5916"
-			(at 276.86 99.9646 90)
+		(property "Value" "TLC5916IPWR"
+			(at 279.4 99.9646 90)
 			(effects
 				(font
@@
 			)
 		)
-		(property "Value" "USB_C_Receptacle_USB2.0_16P"
+		(property "Value" "GT-USB-7070C"
 			(at 33.02 27.94 0)
 			(effects

Commit message: updated models
Parts:
- Q3: footprint Diode_SMD:D_0805_2012Metric -> sw63_mk4:TEMT6200FX01
Changed lines of the file:
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@@
 			)
 		)
-		(property "Footprint" "Diode_SMD:D_0805_2012Metric"
+		(property "Footprint" "sw63_mk4:TEMT6200FX01"
 			(at 116.84 97.79 0)
 			(effects

Commit message: add usb dtct
Parts:
- added R15, R16: 22k, Resistor_SMD:R_0402_1005Metric, symbol Device:R
- R10, R9: value 4k7 -> 5k1
Connections:
- net GND: now also R16.2
- net VBUS: now also R15.1
- net USB_DTCT: now reaches U7.25 (PA15)
- net USB_DTCT: now also R15.2, R16.1
