File: pcb/sw63_mk4_v1/sw63_mk4_v1.kicad_sch (KiCad schematic)
At the start: 70 parts, among them J1 GT-USB-7070C, J2 SWD, J3 Conn_01x02, Q1 DMG2305UX-7, Q2 DMG2302U-7, Q3 TEMT6200FX01, SW1 KSC321J LFS, SW2 ﻿EVQ-P7J01P, U1 DIO5518BST5, U2 MCP1711T-3.3I/OT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

Commit message: bug note
Other:
- note added: "invalid package: 2 and 3 must be swapped"
Changed lines of the file:
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@@
+		)
+	)
+	(text "invalid package: 2 and 3 must be swapped"
+		(exclude_from_sim no)
+		(at 196.342 137.668 0)
+		(effects
+			(font
+				(size 1.27 1.27)
+				(thickness 0.1588)
+			)
 		)
 	)
