File: pcb/sw63_mk4_v2/sw63_mk4_v2.kicad_pcb (KiCad board)
At the start: 4 copper layers, 34.8 x 35.6 mm, 70 parts, among them J1 GT-USB-7070C, J2 SWD, J3 Conn_01x02, Q1 DMG2305UX-7, Q2 DMG2302U-7, Q3 TEMT6200FX01, SW1 KSC321J LFS, SW2 ﻿EVQ-P7J01P, U1 DIO5518BST5, U2 MCP1711T-3.3I/OT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

Commit message: update part names and docs
Parts:
- D1, D10, D11, D12, D2, D3, D4, D5, D6, D7, D8, D9: value LED -> XL-3216UWC
- D13: value LED -> L-53SYDK (Yellow)
- D14: value LED -> LL-504BD2E-B4-2B (Blue)
- D15: value LED -> LL-504PGD2E-G5-2B (Green)
- D16: value LED -> LL-503VD2E-V1-4D (Red)
- D17, D18, D19, D20: value LED -> LL-234YD2Q-1B (Yellow)
- D21: value LED -> FYL-3014LRD1A (Red)
